Commit message: robot_barista: multiple robot spawn rick and morty robot name

File: xacro/barista_robot_model.urdf.xacro (robot description, xacro)
@@ -2,4 +2,5 @@
 <robot xmlns:xacro="http://www.ros.org/wiki/xacro" name="barista_robot">
     <xacro:arg name="include_laser" default="true"/>
+    <xacro:property name="robot_name" value="$(arg robot_name)"/>
     <xacro:include filename="$(find barista_robot_description)/xacro/wheel.xacro" />
     <xacro:include filename="$(find barista_robot_description)/xacro/standoff.xacro" />
@@ -49,18 +50,31 @@
     <gazebo>
         <plugin filename="libgazebo_ros_diff_drive.so" name="differential_drive_controller">
-        <!-- wheels -->
-        <left_joint>wheel_left_chassis_link_joint</left_joint>
-        <right_joint>wheel_right_chassis_link_joint</right_joint>
-        <!-- kinematics -->
-        <wheel_separation>0.266</wheel_separation>
-        <wheel_diameter>0.0704</wheel_diameter>
-        <!-- limits -->
-        <max_wheel_torque>1.0</max_wheel_torque>
-        <max_wheel_acceleration>2.0</max_wheel_acceleration>
-        <!-- output -->
-        <publish_odom>true</publish_odom>
-        <publish_odom_tf>true</publish_odom_tf>
-        <odometry_frame>odom</odometry_frame>
-        <robot_base_frame>base_link</robot_base_frame>
+            <ros>
+                <namespace>/${robot_name}</namespace>
+                <remapping>/cmd_vel:=cmd_vel</remapping>
+            </ros>
+            <!-- wheels -->
+            <left_joint>wheel_left_chassis_link_joint</left_joint>
+            <right_joint>wheel_right_chassis_link_joint</right_joint>
+            <!-- kinematics -->
+            <wheel_separation>0.266</wheel_separation>
+            <wheel_diameter>0.0704</wheel_diameter>
+            <!-- limits -->
+            <max_wheel_torque>1.0</max_wheel_torque>
+            <max_wheel_acceleration>2.0</max_wheel_acceleration>
+            <!-- output -->
+            <publish_odom>true</publish_odom>
+            <publish_odom_tf>true</publish_odom_tf>
+            <odometry_frame>${robot_name}/odom</odometry_frame>>
+            <robot_base_frame>${robot_name}/base_link</robot_base_frame>
+        </plugin>
+        <plugin name="box_bot_joint_state" filename="libgazebo_ros_joint_state_publisher.so">
+            <ros>
+                <namespace>/${robot_name}</namespace>
+                <remapping>~/out:=joint_states</remapping>
+            </ros>
+            <update_rate>30</update_rate>
+            <joint_name>wheel_left_chassis_link_joint</joint_name>
+            <joint_name>wheel_right_chassis_link_joint</joint_name>
         </plugin>
     </gazebo>

File: xacro/laser_scanner.xacro (robot description, xacro)
@@ -76,4 +76,5 @@
                 <plugin name="laser" filename="libgazebo_ros_ray_sensor.so">
                 <ros>
+                    <namespace>/${robot_name}</namespace>
                     <remapping>~/out:=scan</remapping>
                 </ros>
